Commit message: Prokop: CRS93 simulation package, tests, robot measurement tools
- switch from CRS97 to CRS93 (ctu_crs.CRS93): models/crs93.urdf with the
  CRS93 joint limits, CRS93Sim; project renamed crs97 -> crs93
- restructure: URDFs + meshes in models/, generators in tools/
- simulation.CRS93Sim: drop-in for ctu_crs.CRS93 in the Viser scene; kinematics
  are ctu_crs's own (no IK helpers; kinematics.py and freehand IK removed)
- measured table height, camera work area, base foam; cage (CAGE_XY) and spin
  period are placeholders; random placement in the cage, viable placement in
  the camera work area
- hoop: both faces coloured (groove floors blue)
- pytest suite (Prokop/tests): shapes, joint-limit edge cases, sim interface
- tools/log_motion.py (no homing) and tools/camera_survey.py (camera timing,
  image delay) for measurements on the real robot; ROBOT_CHECKS.md, NOTIFY.md
- deps: pytest (dev), opencv-contrib-python

Co-Authored-By: Claude Opus 5.5 (1M context) <noreply@anthropic.com>

File: Prokop/models/base.urdf (robot description, URDF)
Before this commit: robot base, 4 links, 3 joints
Links:
- added link foam; collision box size=0.125 0.125 0.025; visual box size=0.125 0.125 0.025
Joints:
- added joint base_link_to_foam: type fixed, parent base_link, child foam, origin xyz=0 0 0 rpy=0 0 0

File: Prokop/models/crs93.urdf (robot description, URDF)
Before this commit: robot crs97, 10 links, 9 joints
Links:
- link base_link: geometry collision mesh filename=meshes/crs93/link0.stl; visual mesh filename=meshes/crs93/link0.stl
- link link1: geometry collision mesh filename=meshes/crs93/link1.stl; visual mesh filename=meshes/crs93/link1.stl
- link link2: geometry collision mesh filename=meshes/crs93/link2.stl; visual mesh filename=meshes/crs93/link2_0.stl
- link link3: geometry collision mesh filename=meshes/crs93/link3.stl; visual mesh filename=meshes/crs93/link3.stl
- link link4: geometry collision mesh filename=meshes/crs93/link4.stl; visual mesh filename=meshes/crs93/link4.stl
- link link5: geometry collision mesh filename=meshes/crs93/link5.stl; visual mesh filename=meshes/crs93/link5.stl
- link link6: geometry collision mesh filename=meshes/crs93/link6.stl; visual mesh filename=meshes/crs93/link6.stl
Joints:
- joint joint1: limit lower=-2.94524311274 upper=3.02378292908 effort=100 velocity=1.0 -> lower=-2.95859488152 upper=3.0104311603 effort=100 velocity=1.0
- joint joint2: limit lower=-1.57475473354 upper=1.56683792005 effort=100 velocity=1.0 -> lower=-1.56531424761 upper=1.57627840598 effort=100 velocity=1.0
- joint joint3: limit lower=-2.02043677534 upper=1.98509385799 effort=100 velocity=1.0 -> lower=-1.96663700115 upper=2.00747770564 effort=100 velocity=1.0
- joint joint4: limit lower=-3.19758143355 upper=3.24112826242 effort=100 velocity=1.0 -> lower=-3.24423875019 upper=3.24112826242 effort=100 velocity=1.0
- joint joint5: limit lower=-1.81269896112 upper=1.83154851704 effort=100 velocity=1.0 -> lower=-1.84411488766 upper=1.83154851704 effort=100 velocity=1.0
- joint joint6: limit lower=-3.17736326301 upper=3.15247936081 effort=100 velocity=1.0 -> lower=-3.14470314137 upper=3.20380240911 effort=100 velocity=1.0

File: Prokop/models/turntable.urdf (robot description, URDF)
Before this commit: robot turntable, 2 links, 1 joints
Links:
- link turntable_link: geometry collision cylinder length=0.034 radius=0.0685; visual cylinder length=0.034 radius=0.0685
Joints:
- joint turntable_link_to_top: origin xyz=0 0 0.045 -> xyz=0 0 0.034
