Commit message: Prokop: work cell model, collision checks, robot test results
- cell.py: measured table (25 mm below the robot foot top), work area, octagonal
  cage, camera rail + post, camera (Basler a2A1920-51gcBAS, estimated 17 mm lens)
- collision.py: arm + hoop clearance to the table and cell, per pose and path
- adapter turned by 180 deg on the CRS93 station: hoop points up in q_home
  (ADAPTER_TURN in robodk2urdf.py, models/crs93.urdf)
- sim hard home ends at the measured encoder-zero pose; turntable period 28.0 s
- log_motion.py: queued blending tests (corner, reversal, via chains), --tests
- camera_survey.py --delay: checked survey pose with the hoop in view, slow swing
- ROBOT_CHECKS.md: results of the first robot runs and the next runs

Co-Authored-By: Claude Opus 5.5 <noreply@anthropic.com>

File: Prokop/models/crs93.urdf (robot description, URDF)
Before this commit: robot crs93, 10 links, 9 joints
Joints:
- joint flange_to_adapter: origin xyz=0 0 0.002 rpy=3.14159265359 -0 -1.57079632679 -> xyz=0 0 0.002 rpy=3.14159265359 -0 1.57079632679
